Commit message: train with data 1504

File: simulation/Spot1504/urdf/Spot1504.urdf (robot description, URDF)
Before this commit: robot Spot, 17 links, 16 joints
Links:
- removed link chasiss
- added link BASE, mass 5; collision mesh filename=package://Spot1504/meshes/BASE.STL; visual mesh filename=package://Spot1504/meshes/BASE.STL
- link BL_lower_hip: mass 0.1 -> 0.2; geometry collision mesh filename=package://Spot1504/meshes/BL_lower_hip.STL; visual mesh filename=package://Spot1504/meshes/BL_lower_hip.STL
- link BL_lower_knee: mass 0.1 -> 0.2; geometry collision mesh filename=package://Spot1504/meshes/BL_lower_knee.STL; visual mesh filename=package://Spot1504/meshes/BL_lower_knee.STL
- link BL_upper_hip: mass 0.1 -> 0.2; geometry collision mesh filename=package://Spot1504/meshes/BL_upper_hip.STL; visual mesh filename=package://Spot1504/meshes/BL_upper_hip.STL
- link BL_upper_knee: mass 0.1 -> 0.2; geometry collision mesh filename=package://Spot1504/meshes/BL_upper_knee.STL; visual mesh filename=package://Spot1504/meshes/BL_upper_knee.STL
- link BR_lower_hip: mass 0.1 -> 0.2; geometry collision mesh filename=package://Spot1504/meshes/BR_lower_hip.STL; visual mesh filename=package://Spot1504/meshes/BR_lower_hip.STL
- link BR_lower_knee: mass 0.1 -> 0.2; geometry collision mesh filename=package://Spot1504/meshes/BR_lower_knee.STL; visual mesh filename=package://Spot1504/meshes/BR_lower_knee.STL
- link BR_upper_hip: mass 0.1 -> 0.2; geometry collision mesh filename=package://Spot1504/meshes/BR_upper_hip.STL; visual mesh filename=package://Spot1504/meshes/BR_upper_hip.STL
- link BR_upper_knee: mass 0.1 -> 0.2; geometry collision mesh filename=package://Spot1504/meshes/BR_upper_knee.STL; visual mesh filename=package://Spot1504/meshes/BR_upper_knee.STL
- link FL_lower_hip: mass 0.1 -> 0.2; geometry collision mesh filename=package://Spot1504/meshes/FL_lower_hip.STL; visual mesh filename=package://Spot1504/meshes/FL_lower_hip.STL
- link FL_lower_knee: mass 0.1 -> 0.2; geometry collision mesh filename=package://Spot1504/meshes/FL_lower_knee.STL; visual mesh filename=package://Spot1504/meshes/FL_lower_knee.STL
- link FL_upper_hip: mass 0.1 -> 0.2; geometry collision mesh filename=package://Spot1504/meshes/FL_upper_hip.STL; visual mesh filename=package://Spot1504/meshes/FL_upper_hip.STL
- link FL_upper_knee: mass 0.1 -> 0.2; geometry collision mesh filename=package://Spot1504/meshes/FL_upper_knee.STL; visual mesh filename=package://Spot1504/meshes/FL_upper_knee.STL
- link FR_lower_hip: mass 0.1 -> 0.2; geometry collision mesh filename=package://Spot1504/meshes/FR_lower_hip.STL; visual mesh filename=package://Spot1504/meshes/FR_lower_hip.STL
- link FR_lower_knee: mass 0.1 -> 0.2; geometry collision mesh filename=package://Spot1504/meshes/FR_lower_knee.STL; visual mesh filename=package://Spot1504/meshes/FR_lower_knee.STL
- link FR_upper_hip: mass 0.1 -> 0.2; geometry collision mesh filename=package://Spot1504/meshes/FR_upper_hip.STL; visual mesh filename=package://Spot1504/meshes/FR_upper_hip.STL
- link FR_upper_knee: mass 0.1 -> 0.2; geometry collision mesh filename=package://Spot1504/meshes/FR_upper_knee.STL; visual mesh filename=package://Spot1504/meshes/FR_upper_knee.STL
Joints:
- joint bl_lower_hip_joint: origin xyz=-0.097481 0.01 -0.050966 rpy=0 0 0 -> xyz=-0.1035 0.01 -0.037254 rpy=0 0 0
- joint bl_lower_knee_joint: origin xyz=0.086726 0.008 -0.067666 rpy=0 0 0 -> xyz=0.0800840565833425 0.00799999999999989 -0.0754091763723482 rpy=0 0 0
- joint br_lower_hip_joint: origin xyz=-0.097481 -0.01 -0.050966 rpy=0 0 0 -> xyz=-0.103499423252635 -0.0100000000000007 -0.0372541190514647 rpy=0 0 0
- joint br_lower_knee_joint: origin xyz=0.086726 -0.008 -0.067666 rpy=0 0 0 -> xyz=0.0800840565833414 -0.00800000000000095 -0.0754091763723471 rpy=0 0 0
- joint fl_lower_hip_joint: origin xyz=-0.097481 0.01 -0.050966 rpy=0 0 0 -> xyz=-0.103501820756454 0.0100000000000031 -0.0372474576318325 rpy=0 0 0
- joint fl_lower_knee_joint: origin xyz=0.086726 0.008 -0.067666 rpy=0 0 0 -> xyz=0.0800874913210537 0.00799999999999891 -0.0754055285368097 rpy=0 0 0
- joint fr_lower_hip_joint: origin xyz=-0.097594 -0.01 -0.050749 rpy=0 0 0 -> xyz=-0.103501820756658 -0.010000000000002 -0.0372474576320085 rpy=0 0 0
- joint fr_lower_knee_joint: origin xyz=0.086649 -0.008 -0.067764 rpy=0 0 0 -> xyz=0.080087 -0.008 -0.075406 rpy=0 0 0
- joint motor_bl_upper_hip_joint: origin xyz=-0.24756 0.1735 0.007712 rpy=0 0 0 -> xyz=-0.246888764816589 0.173499648835901 0.00749192202401183 rpy=0 0 0; parent chasiss -> BASE
- joint motor_bl_upper_knee_joint: origin xyz=-0.19756 0.1735 0.007712 rpy=0 0 0 -> xyz=-0.196888764816585 0.173499648835901 0.00749192202401999 rpy=0 0 0; parent chasiss -> BASE
- joint motor_br_upper_hip_joint: origin xyz=-0.24756 -0.1735 0.007712 rpy=0 0 0 -> xyz=-0.246888764816864 -0.173500351164099 0.00749192202338655 rpy=0 0 0; parent chasiss -> BASE
- joint motor_br_upper_knee_joint: origin xyz=-0.19756 -0.1735 0.007712 rpy=0 0 0 -> xyz=-0.196888764816585 -0.173500351164099 0.00749192202402094 rpy=0 0 0; parent chasiss -> BASE
- joint motor_fl_upper_hip_joint: origin xyz=0.19844 0.1735 0.007712 rpy=0 0 0 -> xyz=0.199111235183205 0.173499648835901 0.00749192202384069 rpy=0 0 0; parent chasiss -> BASE
- joint motor_fl_upper_knee_joint: origin xyz=0.24844 0.1735 0.007712 rpy=0 0 0 -> xyz=0.249111235183415 0.173499648835901 0.0074919220240201 rpy=0 0 0; parent chasiss -> BASE
- joint motor_fr_upper_hip_joint: origin xyz=0.19775 -0.1735 0.0069919 rpy=0 0 0 -> xyz=0.19911123518341 -0.173500351164098 0.00749192202401805 rpy=0 0 0; parent chasiss -> BASE
- joint motor_fr_upper_knee_joint: origin xyz=0.24844 -0.1735 0.007712 rpy=0 0 0 -> xyz=0.24911 -0.1735 0.0074919 rpy=0 0 0; parent chasiss -> BASE

Commit message: ready for training

File: simulation/Spot1504/urdf/Spot1504.urdf (robot description, URDF)
Before this commit: robot Spot1504, 17 links, 16 joints
Links:
- link BASE: mass 5 -> 7
